File: Qwerty/qwerty.kicad_sch (KiCad schematic)
At the start: 84 parts, among them J1 Conn_01x16, J2 Conn_01x10, J3 J, K1 K, M1 M, P1 P, Q1 Q, SW1 SW_DIP_x01, T1 T, U1 U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

Commit message: Setup 3D models on PCB for connectors
Parts:
- J1: footprint AS_Parts:SLW16R-1C7LF -> SLW16R-1C7LF:CON16_1X16_RB_58JF_GLE
- J2: footprint AS_Parts:HLW10R-2C7LF -> HLW10R-2C7LF:AMPHENOL_HLW10R-2C7LF
