File: Qwerty/qwerty.kicad_pcb (KiCad board)
At the start: 2 copper layers, 276 x 133 mm, 95 parts, among them J1 Conn_01x16, J2 Conn_01x10, J3 J, K1 K, M1 M, P1 P, Q1 Q, SW1 SW_DIP_x01, T1 T, U1 U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

Commit message: Updated kicad and gerbers to latest version of kicad
Other:
- net class Default removed

Commit message: Setup 3D models on PCB for connectors
Parts:
- added REF**: CON16_1X16_RB_58JF_GLE, SLW16R-1C7LF:CON16_1X16_RB_58JF_GLE, B.Cu at (204.4, 65.6)
- added REF**: AMPHENOL_HLW10R-2C7LF, HLW10R-2C7LF:AMPHENOL_HLW10R-2C7LF, B.Cu at (229.9, 61.0)

Commit message: Updated connector footprint on PCB
Parts:
- removed the REF** at (204.4, 65.6)
- removed the REF** at (229.9, 61.0)
- J1: footprint AS_Parts:SLW16R-1C7LF -> SLW16R-1C7LF:CON16_1X16_RB_58JF_GLE
- J2: footprint AS_Parts:HLW10R-2C7LF -> HLW10R-2C7LF:AMPHENOL_HLW10R-2C7LF
- moved J1 7.58 mm to (204.5, 76.5), turned to 180 degrees
- moved J2 1.58 mm to (228.9, 73.9)
Connections:
- J1 pad 1: /COL1 -> /COL16
- J1 pad 10: /COL10 -> /COL7
- J1 pad 11: /COL11 -> /COL6
- J1 pad 12: /COL12 -> /COL5
- J1 pad 13: /COL13 -> /COL4
- J1 pad 14: /COL14 -> /COL3
- J1 pad 15: /COL15 -> /COL2
- J1 pad 16: /COL16 -> /COL1
- J1 pad 2: /COL2 -> /COL15
- J1 pad 3: /COL3 -> /COL14
- J1 pad 4: /COL4 -> /COL13
- J1 pad 5: /COL5 -> /COL12
- J1 pad 6: /COL6 -> /COL11
- J1 pad 7: /COL7 -> /COL10
- J1 pad 8: /COL8 -> /COL9
- J1 pad 9: /COL9 -> /COL8
